Commit message: last version
Signed-off-by: Tomas Lorente <jtlorente@ekumenlabs.com>

File: cheetah_gym/urdf/mini_cheetah.urdf (robot description, URDF)
Before this commit: robot mini_cheetah, 17 links, 16 joints
Links:
- link abduct_fl: geometry collision mesh filename=/home/cheetah_gym/cheetah_gym/urdf/meshes/mini_abad.dae; visual mesh filename=/home/cheetah_gym/cheetah_gym/urdf/meshes/mini_abad.dae
- link abduct_fr: geometry collision mesh filename=/home/cheetah_gym/cheetah_gym/urdf/meshes/mini_abad.dae; visual mesh filename=/home/cheetah_gym/cheetah_gym/urdf/meshes/mini_abad.dae
- link abduct_hl: geometry collision mesh filename=/home/cheetah_gym/cheetah_gym/urdf/meshes/mini_abad.dae; visual mesh filename=/home/cheetah_gym/cheetah_gym/urdf/meshes/mini_abad.dae
- link abduct_hr: geometry collision mesh filename=/home/cheetah_gym/cheetah_gym/urdf/meshes/mini_abad.dae; visual mesh filename=/home/cheetah_gym/cheetah_gym/urdf/meshes/mini_abad.dae
- link body: geometry collision mesh filename=/home/cheetah_gym/cheetah_gym/urdf/meshes/mini_body.dae; visual mesh filename=/home/cheetah_gym/cheetah_gym/urdf/meshes/mini_body.dae
- link shank_fl: geometry collision mesh filename=/home/cheetah_gym/cheetah_gym/urdf/meshes/mini_lower_link.d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; visual mesh filename=/home/cheetah_gym/cheetah_gym/urdf/meshes/mini_lower_link.d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
- link shank_fr: geometry collision mesh filename=/home/cheetah_gym/cheetah_gym/urdf/meshes/mini_lower_link.d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; visual mesh filename=/home/cheetah_gym/cheetah_gym/urdf/meshes/mini_lower_link.d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
- link shank_hl: geometry collision mesh filename=/home/cheetah_gym/cheetah_gym/urdf/meshes/mini_lower_link.d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; visual mesh filename=/home/cheetah_gym/cheetah_gym/urdf/meshes/mini_lower_link.d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
- link shank_hr: geometry collision mesh filename=/home/cheetah_gym/cheetah_gym/urdf/meshes/mini_lower_link.d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; visual mesh filename=/home/cheetah_gym/cheetah_gym/urdf/meshes/mini_lower_link.d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
- link thigh_fl: geometry collision mesh filename=/home/cheetah_gym/cheetah_gym/urdf/meshes/mini_upper_link.d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; visual mesh filename=/home/cheetah_gym/cheetah_gym/urdf/meshes/mini_upper_link.d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
- link thigh_fr: geometry collision mesh filename=/home/cheetah_gym/cheetah_gym/urdf/meshes/mini_upper_link.d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; visual mesh filename=/home/cheetah_gym/cheetah_gym/urdf/meshes/mini_upper_link.d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
- link thigh_hl: geometry collision mesh filename=/home/cheetah_gym/cheetah_gym/urdf/meshes/mini_upper_link.d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; visual mesh filename=/home/cheetah_gym/cheetah_gym/urdf/meshes/mini_upper_link.d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
- link thigh_hr: geometry collision mesh filename=/home/cheetah_gym/cheetah_gym/urdf/meshes/mini_upper_link.d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; visual mesh filename=/home/cheetah_gym/cheetah_gym/urdf/meshes/mini_upper_link.d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

Commit message: updated to baselines
Signed-off-by: Lobotuerk <tomas.lobo.it@gmail.com>

File: cheetah_gym/urdf/mini_cheetah.urdf (robot description, URDF)
Before this commit: robot mini_cheetah, 17 links, 16 joints
Links:
- link abduct_fl: geometry collision mesh filename=meshes/mini_abad.dae; visual mesh filename=meshes/mini_abad.dae
- link abduct_fr: geometry collision mesh filename=meshes/mini_abad.dae; visual mesh filename=meshes/mini_abad.dae
- link abduct_hl: geometry collision mesh filename=meshes/mini_abad.dae; visual mesh filename=meshes/mini_abad.dae
- link abduct_hr: geometry collision mesh filename=meshes/mini_abad.dae; visual mesh filename=meshes/mini_abad.dae
- link body: geometry collision mesh filename=meshes\mini_body.dae; visual mesh filename=meshes\mini_body.dae
- link shank_fl: geometry collision mesh filename=meshes/mini_lower_link_no_toe.dae; visual mesh filename=meshes/mini_lower_link.dae
- link shank_fr: geometry collision mesh filename=meshes/mini_lower_link_no_toe.dae; visual mesh filename=meshes/mini_lower_link.dae
- link shank_hl: geometry collision mesh filename=meshes/mini_lower_link_no_toe.dae; visual mesh filename=meshes/mini_lower_link.dae
- link shank_hr: geometry collision mesh filename=meshes/mini_lower_link_no_toe.dae; visual mesh filename=meshes/mini_lower_link.dae
- link thigh_fl: geometry collision mesh filename=meshes/mini_upper_link.dae; visual mesh filename=meshes/mini_upper_link.dae
- link thigh_fr: geometry collision mesh filename=meshes/mini_upper_link.dae; visual mesh filename=meshes/mini_upper_link.dae
- link thigh_hl: geometry collision mesh filename=meshes/mini_upper_link.dae; visual mesh filename=meshes/mini_upper_link.dae
- link thigh_hr: geometry collision mesh filename=meshes/mini_upper_link.dae; visual mesh filename=meshes/mini_upper_link.dae

Commit message: update_ekumen
Signed-off-by: tomas.plusone <jtlorente@creativa77.com.ar>

File: cheetah_gym/urdf/mini_cheetah.urdf (robot description, URDF)
Before this commit: robot mini_cheetah, 17 links, 16 joints
Links:
- link body: geometry collision mesh filename=meshes/mini_body.dae; visual mesh filename=meshes/mini_body.dae
